File: SensebenderMicro2.sch (KiCad schematic (older format))
At the start: 41 parts, among them P2 MYSX_2.4, P3 Antenna, Q1 SI2333DDS-T1-GE3, U1 ATSAMD21E, U2 MCP1703T-3302E, U3 NRF24L01, U4 RFM69HW, U5 ATSHA204A, U6 AT45DB041E, U7 Si7021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

Commit message: Updated routing, gnd on component side
Parts:
- removed Q1: SI2333DDS-T1-GE3, TO_SOT_Packages_SMD:SOT-23, symbol Q_NMOS_GSD
- removed R7: 100K, Resistors_SMD:R_0603, symbol R
- added D3: LED, LEDs:LED-0603, symbol LED
- P3: symbol CONN_01X01 -> CONN_01X02
- R6: value 100R -> 220R
Connections:
- net +3.3VP is gone; now on net +3V3: C11.1, C9.2, U3.2 (VCC), U4.8 (3.3V)
- net GND: now also P3.2 (P2), D3.1 (K)
- net at U1.27 (PA28): now also R6.1; no longer R6.2
- new net: D3.2 (A), R6.2
Other:
- note removed: "Q1 opens when Gate is held low. \nSo we have a resistor pulling the \ngate high, to disable the radio by\ndefault.\n\nIf we had the resistor to gnd, and \nthus have the radio to be default on,\nwe had to take the current draw through\nR7 into account, whenever we wanted to\npower down the radios."
Changed lines of the file:
@@
 D8_SDA
 $Comp
-L CONN_01X01 P3
+L CONN_01X02 P3
 U 1 1 56B7B00E
-P 7750 950
-F 0 "P3" H 7750 1050 50  0000 C CNN
-F 1 "Antenna" V 7850 950 50  0000 C CNN
-F 2 "Pin_Headers:Pin_Header_Straight_1x01" H 7750 950 50  0001 C CNN
-F 3 "" H 7750 950 50  0000 C CNN
-	1    7750 950
+P 7800 950
+F 0 "P3" H 7800 1050 50  0000 C CNN
+F 1 "Antenna" V 7900 950 50  0000 C CNN
+F 2 "Pin_Headers:Pin_Header_Straight_1x01" H 7800 950 50  0001 C CNN
+F 3 "" H 7800 950 50  0000 C CNN
+	1    7800 950
 	0    -1   -1   0
 $EndComp
@@
 $EndComp
 $Comp
-L Q_NMOS_GSD Q1
-U 1 1 571F69BC
-P 6400 4800
-F 0 "Q1" V 6550 4700 50  0000 R CNN
-F 1 "SI2333DDS-T1-GE3" V 6400 4600 50  0000 R CNN
-F 2 "TO_SOT_Packages_SMD:SOT-23" H 6600 4900 50  0001 C CNN
-F 3 "" H 6400 4800 50  0000 C CNN
-	1    6400 4800
-	0    -1   -1   0
-$EndComp
-$Comp
-L +3.3VP #PWR032
-U 1 1 571F74A2
-P 8550 900
-F 0 "#PWR032" H 8700 850 50  0001 C CNN
-F 1 "+3.3VP" H 8570 1043 50  0000 C CNN
-F 2 "" H 8550 900 50  0000 C CNN
-F 3 "" H 8550 900 50  0000 C CNN
-	1    8550 900
-	1    0    0    -1
-$EndComp
-$Comp
-L +3.3VP #PWR033
-U 1 1 571F74FA
-P 10000 1000
-F 0 "#PWR033" H 10150 950 50  0001 C CNN
-F 1 "+3.3VP" H 10020 1143 50  0000 C CNN
-F 2 "" H 10000 1000 50  0000 C CNN
-F 3 "" H 10000 1000 50  0000 C CNN
-	1    10000 1000
-	1    0    0    -1
-$EndComp
-$Comp
-L +3.3VP #PWR034
-U 1 1 571F77CE
-P 6650 4600
-F 0 "#PWR034" H 6800 4550 50  0001 C CNN
-F 1 "+3.3VP" H 6670 4743 50  0000 C CNN
-F 2 "" H 6650 4600 50  0000 C CNN
-F 3 "" H 6650 4600 50  0000 C CNN
-	1    6650 4600
-	1    0    0    -1
-$EndComp
-$Comp
-L +3V3 #PWR035
-U 1 1 571F7898
-P 6150 4600
-F 0 "#PWR035" H 6150 4450 50  0001 C CNN
-F 1 "+3V3" H 6165 4773 50  0000 C CNN
-F 2 "" H 6150 4600 50  0000 C CNN
-F 3 "" H 6150 4600 50  0000 C CNN
-	1    6150 4600
-	1    0    0    -1
-$EndComp
-$Comp
 L JUMPER3 JP1
 U 1 1 5725B163
@@
 $EndComp
 $Comp
-L +3V3 #PWR036
+L +3V3 #PWR034
 U 1 1 5726438E
 P 8300 2900
-F 0 "#PWR036" H 8300 2750 50  0001 C CNN
+F 0 "#PWR034" H 8300 2750 50  0001 C CNN
 F 1 "+3V3" H 8315 3073 50  0000 C CNN
 F 2 "" H 8300 2900 50  0000 C CNN
@@
 	1    8300 2900
 	1    0    0    -1
-$EndComp
-$Comp
-L R R6
-U 1 1 57279B05
-P 5550 5850
-F 0 "R6" V 5343 5850 50  0000 C CNN
-F 1 "100R" V 5434 5850 50  0000 C CNN
-F 2 "Resistors_SMD:R_0603" V 5480 5850 50  0001 C CNN
-F 3 "" H 5550 5850 50  0000 C CNN
-	1    5550 5850
-	0    1    1    0
 $EndComp
 Wire Wire Line
@@
 Connection ~ 2300 2900
 Wire Wire Line
-	6400 5000 6400 5850
-Wire Wire Line
-	6600 4700 6650 4700
-Wire Wire Line
-	6650 4700 6650 4600
-Wire Wire Line
-	6150 4600 6150 4700
-Wire Wire Line
-	6150 4700 6200 4700
-Wire Wire Line
 	9900 5050 9900 5100
 Wire Wire Line
@@
 	8850 5200 9650 5200
 Connection ~ 8850 5600
-Wire Wire Line
-	6400 5850 5700 5850
-$Comp
-L +3V3 #PWR037
-U 1 1 5727A1DE
-P 6050 5450
-F 0 "#PWR037" H 6050 5300 50  0001 C CNN
-F 1 "+3V3" H 6065 5623 50  0000 C CNN
-F 2 "" H 6050 5450 50  0000 C CNN
-F 3 "" H 6050 5450 50  0000 C CNN
-	1    6050 5450
-	1    0    0    -1
-$EndComp
-$Comp
-L R R7
-U 1 1 5727A23C
-P 6050 5650
-F 0 "R7" H 6120 5696 50  0000 L CNN
-F 1 "100K" H 6120 5605 50  0000 L CNN
-F 2 "Resistors_SMD:R_0603" V 5980 5650 50  0001 C CNN
-F 3 "" H 6050 5650 50  0000 C CNN
-	1    6050 5650
-	1    0    0    -1
-$EndComp
-Wire Wire Line
-	6050 5800 6050 5850
-Connection ~ 6050 5850
-Text Notes 6500 5900 0    60   ~ 0
-Q1 opens when Gate is held low. \nSo we have a resistor pulling the \ngate high, to disable the radio by\ndefault.\n\nIf we had the resistor to gnd, and \nthus have the radio to be default on,\nwe had to take the current draw through\nR7 into account, whenever we wanted to\npower down the radios.
 Wire Wire Line
 	10300 5200 10300 5600
@@
 Connection ~ 10000 1050
 $Comp
-L GND #PWR038
+L GND #PWR035
 U 1 1 5761A76F
 P 9600 1100
-F 0 "#PWR038" H 9600 850 50  0001 C CNN
+F 0 "#PWR035" H 9600 850 50  0001 C CNN
 F 1 "GND" H 9605 927 50  0000 C CNN
 F 2 "" H 9600 1100 50  0000 C CNN
@@
 Wire Wire Line
 	9850 4250 10100 4250
-Wire Wire Line
-	6050 5450 6050 5500
 Wire Wire Line
 	9850 5900 9850 5950
@@
 LEGACY_ID
 $Comp
-L +3.3VA #PWR039
+L +3.3VA #PWR036
 U 1 1 5828CA22
 P 2300 2900
-F 0 "#PWR039" H 2300 2750 50  0001 C CNN
+F 0 "#PWR036" H 2300 2750 50  0001 C CNN
 F 1 "+3.3VA" H 2315 3073 50  0000 C CNN
 F 2 "" H 2300 2900 50  0000 C CNN
@@
 Wire Wire Line
 	3600 5950 4700 5950
-Wire Wire Line
-	3600 6050 5400 6050
-Wire Wire Line
-	5400 6050 5400 5850
 Wire Wire Line
 	1500 6650 2500 6650
@@
 $EndComp
 $Comp
-L +3V3 #PWR040
+L +3V3 #PWR037
 U 1 1 582A3CE8
 P 950 6650
-F 0 "#PWR040" H 950 6500 50  0001 C CNN
+F 0 "#PWR037" H 950 6500 50  0001 C CNN
 F 1 "+3V3" H 965 6823 50  0000 C CNN
 F 2 "" H 950 6650 50  0000 C CNN
@@
 $EndComp
 $Comp
-L +3V3 #PWR041
+L +3V3 #PWR038
 U 1 1 582F12E3
 P 10200 2900
-F 0 "#PWR041" H 10200 2750 50  0001 C CNN
+F 0 "#PWR038" H 10200 2750 50  0001 C CNN
 F 1 "+3V3" H 10215 3073 50  0000 C CNN
 F 2 "" H 10200 2900 50  0000 C CNN
@@
 Text Label 3600 4350 0    60   ~ 0
 D5_PWM
+$Comp
+L LED D3
+U 1 1 5838D210
+P 5300 6600
+F 0 "D3" H 5300 6700 50  0000 C CNN
+F 1 "LED" H 5300 6500 50  0000 C CNN
+F 2 "LEDs:LED-0603" H 5300 6600 50  0001 C CNN
+F 3 "" H 5300 6600 50  0000 C CNN
+	1    5300 6600
+	0    -1   -1   0
+$EndComp
+$Comp
+L R R6
+U 1 1 5838D216
+P 5300 6250
+F 0 "R6" V 5380 6250 50  0000 C CNN
+F 1 "220R" V 5300 6250 50  0000 C CNN
+F 2 "Resistors_SMD:R_0603" V 5230 6250 50  0001 C CNN
+F 3 "" H 5300 6250 50  0000 C CNN
+	1    5300 6250
+	1    0    0    -1
+$EndComp
+$Comp
+L GND #PWR039
+U 1 1 5838D21C
+P 5300 6800
+F 0 "#PWR039" H 5300 6550 50  0001 C CNN
+F 1 "GND" H 5300 6650 50  0000 C CNN
+F 2 "" H 5300 6800 50  0000 C CNN
+F 3 "" H 5300 6800 50  0000 C CNN
+	1    5300 6800
+	1    0    0    -1
+$EndComp
+Wire Wire Line
+	3600 6050 5300 6050
+Wire Wire Line
+	5300 6050 5300 6100
+$Comp
+L +3.3V #PWR?
+U 1 1 5838DA32
+P 8550 900
+F 0 "#PWR?" H 8550 750 50  0001 C CNN
+F 1 "+3.3V" H 8565 1073 50  0000 C CNN
+F 2 "" H 8550 900 50  0000 C CNN
+F 3 "" H 8550 900 50  0000 C CNN
+	1    8550 900
+	1    0    0    -1
+$EndComp
+$Comp
+L +3.3V #PWR?
+U 1 1 5838DABF
+P 10000 1000
+F 0 "#PWR?" H 10000 850 50  0001 C CNN
+F 1 "+3.3V" H 10015 1173 50  0000 C CNN
+F 2 "" H 10000 1000 50  0000 C CNN
+F 3 "" H 10000 1000 50  0000 C CNN
+	1    10000 1000
+	1    0    0    -1
+$EndComp
+$Comp
+L GND #PWR?
+U 1 1 583B0428
+P 7850 1150
+F 0 "#PWR?" H 7850 900 50  0001 C CNN
+F 1 "GND" V 7855 1022 50  0000 R CNN
+F 2 "" H 7850 1150 50  0000 C CNN
+F 3 "" H 7850 1150 50  0000 C CNN
+	1    7850 1150
+	0    -1   -1   0
+$EndComp
 $EndSCHEMATC
